File: model/EPS32-D1-Mini-Controller/EPS32-D1-Mini-Controller.kicad_sch (KiCad schematic)
At the start: 23 parts, among them J1 Buck Converter, J2 I2C, J3 LED Channel 1, J4 LED Channel 2, J5 LED Channel 3, J6 LED Channel 4, J7 5V/12V Power, J8 I2C, J9 Barrel_Jack, U1 esp32-wemos-d1-mini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

Commit message: fix barrell jack
Connections:
- net +VCC: now also J9.1; no longer J9.2
- net GND: now also J9.2; no longer J9.1

Commit message: updates
Parts:
- J3, J4, J5, J6: footprint Connector_JST:JST_PH_S3B-PH-K_1x03_P2.00mm_Horizontal -> TerminalBlock_Phoenix:TerminalBlock_Phoenix_MPT-0,5-3-2.54_1x03_P2.54mm_Horizontal
Changed lines of the file:
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@@
 			)
 		)
-		(property "Footprint" "Connector_JST:JST_PH_S3B-PH-K_1x03_P2.00mm_Horizontal"
+		(property "Footprint" "TerminalBlock_Phoenix:TerminalBlock_Phoenix_MPT-0,5-3-2.54_1x03_P2.54mm_Horizontal"
 			(at 224.79 83.82 0)
 			(effects
@@
 			)
 		)
-		(property "Footprint" "Connector_JST:JST_PH_S3B-PH-K_1x03_P2.00mm_Horizontal"
+		(property "Footprint" "TerminalBlock_Phoenix:TerminalBlock_Phoenix_MPT-0,5-3-2.54_1x03_P2.54mm_Horizontal"
 			(at 226.06 153.67 0)
 			(effects
@@
 			)
 		)
-		(property "Footprint" "Connector_JST:JST_PH_S3B-PH-K_1x03_P2.00mm_Horizontal"
+		(property "Footprint" "TerminalBlock_Phoenix:TerminalBlock_Phoenix_MPT-0,5-3-2.54_1x03_P2.54mm_Horizontal"
 			(at 224.79 105.41 0)
 			(effects
@@
 			)
 		)
-		(property "Footprint" "Connector_JST:JST_PH_S3B-PH-K_1x03_P2.00mm_Horizontal"
+		(property "Footprint" "TerminalBlock_Phoenix:TerminalBlock_Phoenix_MPT-0,5-3-2.54_1x03_P2.54mm_Horizontal"
 			(at 224.79 127 0)
 			(effects
