File: model/ESP32_SMD/ESP32_SMD.kicad_pcb (KiCad board)
At the start: 2 copper layers, 98.2 x 54.9 mm, 30 parts, among them J1 Buck Converter, J10 Buck Converter, J2 I2C, J3 LED Channel 1, J4 LED Channel 2, J5 LED Channel 3, J6 LED Channel 4, J7 5V/12V24V Power, J8 I2C, J9 Barrel_Jack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

Commit message: updates
Parts:
- removed REF** (x4): MountingHole_2.2mm_M2_DIN965_Pad, MountingHole:MountingHole_2.2mm_M2_DIN965_Pad
- added H1: MountingHole, MountingHole:MountingHole_2.2mm_M2_DIN965_Pad, F.Cu at (121.3, 34.3)
- added H2: MountingHole, MountingHole:MountingHole_2.2mm_M2_DIN965_Pad, F.Cu at (29.2, 34.3)
- added H3: MountingHole, MountingHole:MountingHole_2.2mm_M2_DIN965_Pad, F.Cu at (121.3, 83.2)
- added H4: MountingHole, MountingHole:MountingHole_2.2mm_M2_DIN965_Pad, F.Cu at (29.2, 83.2)
- added J11: Programming, Connector_JST:JST_XH_B4B-XH-A_1x04_P2.50mm_Vertical, F.Cu at (76.3, 79.5)
- added R6: 10k, PCM_Resistor_THT_AKL:R_Axial_DIN0207_L6.3mm_D2.5mm_P10.16mm_Horizontal, F.Cu at (60.3, 76.8)
- added SW2: Boot, Button_Switch_SMD:SW_SPST_PTS647_Sx38, F.Cu at (60.2, 82.5)
- J1: value Buck Converter -> Buck Converter +5V
- J10: value Buck Converter -> Buck Converter +3.3V
- moved SW1 12.1 mm to (50.8, 82.5)
- moved C2 10.4 mm to (31.0, 74.2)
- moved R5 10.2 mm to (47.0, 76.8)
- moved C1 9.09 mm to (37.0, 78.1)
- moved J10 3.48 mm to (36.6, 64.0), turned to 0 degrees
Connections:
- U2 pad 25: unconnected-(U2-GPIO0/BOOT/ADC2_CH1-Pad25) -> +3.3V_BOOT
- U2 pad 34: unconnected-(U2-U0RXD/GPIO3-Pad34) -> RXD
- U2 pad 35: unconnected-(U2-U0TXD/GPIO1-Pad35) -> TXD
Routing:
- net +3.3V: track 147.9 -> 206.6 mm
- net RXD: track 0.00 -> 48.8 mm, vias 0 -> 1
- net +3.3V_BOOT: track 0.00 -> 39.7 mm, vias 0 -> 2
- net TXD: track 0.00 -> 38.8 mm, vias 0 -> 1
- net GND: track 60.2 -> 69.5 mm
- net +3.3V_EN: track 23.4 -> 16.2 mm, vias 0 -> 2
Other:
- board text added: "3.3V"
- board text added: "GND"
- board text added: "RX"
- board text added: "TX"
- board text removed: "+3.3V"
- board text removed: "+5V"

Commit message: updates
Changed lines of the file:
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@@
 	)
 	(gr_text "WLED 4 Channel\nController V 1.0"
-		(at 91.7 77.1 0)
+		(at 60.4 51.5 0)
 		(layer "F.SilkS" knockout)
 		(effects

Commit message: fixed barrel jack
Connections:
- J9 pad 1: GND -> +VCC
- J9 pad 2: +VCC -> GND

Commit message: updates
Parts:
- J3, J4, J5, J6: footprint Connector_JST:JST_PH_S3B-PH-K_1x03_P2.00mm_Horizontal -> TerminalBlock_Phoenix:TerminalBlock_Phoenix_MPT-0,5-3-2.54_1x03_P2.54mm_Horizontal
