File: model/ESP32_SMD/ESP32_SMD.kicad_sch (KiCad schematic)
At the start: 33 parts, among them J1 Buck Converter, J10 Buck Converter, J11 Screw_Terminal_01x04, J2 I2C, J3 LED Channel 1, J4 LED Channel 2, J5 LED Channel 3, J6 LED Channel 4, J7 5V/12V24V Power, J8 I2C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

Commit message: updates
Parts:
- J1: value Buck Converter -> Buck Converter +5V
- J10: value Buck Converter -> Buck Converter +3.3V
- J11: value Screw_Terminal_01x04 -> Programming
- SW2: value Reset -> Boot
Connections:
- net +3.3V: now also R6.1; no longer R6.2
- net +3.3V_BOOT: now also R6.2; no longer R6.1
Other:
- moved on the sheet: R6
Changed lines of the file:
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@@
 	)
 	(junction
-		(at 123.19 83.82)
+		(at 218.44 77.47)
 		(diameter 0)
 		(color 0 0 0 0)
 	)
 	(junction
-		(at 218.44 77.47)
+		(at 121.92 83.82)
 		(diameter 0)
 		(color 0 0 0 0)
 	)
 	(junction
-		(at 121.92 83.82)
+		(at 119.38 83.82)
 		(diameter 0)
 		(color 0 0 0 0)
@@
 	(wire
 		(pts
-			(xy 123.19 72.39) (xy 123.19 83.82)
-		)
-		(stroke
-			(width 0)
-			(type default)
-		)
-	)
-	(wire
-		(pts
 			(xy 38.1 66.04) (xy 36.83 66.04)
 		)
@@
 	(wire
 		(pts
+			(xy 121.92 62.23) (xy 121.92 83.82)
+		)
+		(stroke
+			(width 0)
+			(type default)
+		)
+	)
+	(wire
+		(pts
+			(xy 121.92 83.82) (xy 133.35 83.82)
+		)
+		(stroke
+			(width 0)
+			(type default)
+		)
+	)
+	(wire
+		(pts
 			(xy 118.11 104.14) (xy 102.87 104.14)
 		)
@@
 	(wire
 		(pts
+			(xy 119.38 83.82) (xy 121.92 83.82)
+		)
+		(stroke
+			(width 0)
+			(type default)
+		)
+	)
+	(wire
+		(pts
 			(xy 34.29 142.24) (xy 35.56 142.24)
 		)
@@
 	(wire
 		(pts
-			(xy 102.87 83.82) (xy 121.92 83.82)
+			(xy 102.87 83.82) (xy 119.38 83.82)
 		)
 		(stroke
@@
 	(wire
 		(pts
-			(xy 123.19 83.82) (xy 133.35 83.82)
-		)
-		(stroke
-			(width 0)
-			(type default)
-		)
-	)
-	(wire
-		(pts
 			(xy 24.13 67.31) (xy 24.13 62.23)
 		)
@@
 	(wire
 		(pts
-			(xy 121.92 62.23) (xy 121.92 83.82)
-		)
-		(stroke
-			(width 0)
-			(type default)
-		)
-	)
-	(wire
-		(pts
-			(xy 121.92 83.82) (xy 123.19 83.82)
+			(xy 119.38 66.04) (xy 119.38 83.82)
 		)
 		(stroke
@@
 	(wire
 		(pts
-			(xy 132.08 72.39) (xy 130.81 72.39)
-		)
-		(stroke
-			(width 0)
-			(type default)
-		)
-	)
-	(wire
-		(pts
 			(xy 36.83 66.04) (xy 36.83 76.2)
 		)
@@
 			)
 		)
-		(property "Value" "Screw_Terminal_01x04"
+		(property "Value" "Programming"
 			(at 43.18 139.6999 0)
 			(effects
@@
 			)
 		)
-		(property "Value" "Buck Converter"
+		(property "Value" "Buck Converter +5V"
 			(at 61.468 42.926 90)
 			(effects
@@
 			)
 		)
-		(property "Value" "Reset"
+		(property "Value" "Boot"
 			(at 127 58.42 0)
 			(effects
@@
 			)
 		)
-		(property "Value" "Buck Converter"
+		(property "Value" "Buck Converter +3.3V"
 			(at 89.408 44.196 90)
 			(effects
@@
 	(symbol
 		(lib_id "Device:R")
-		(at 127 72.39 90)
+		(at 115.57 66.04 90)
 		(unit 1)
 		(exclude_from_sim no)
@@
 		(dnp no)
 		(property "Reference" "R6"
-			(at 127 75.438 90)
+			(at 115.57 69.088 90)
 			(effects
 				(font
@@
 		)
 		(property "Value" "10k"
-			(at 126.746 69.088 90)
+			(at 115.316 62.738 90)
 			(effects
 				(font
@@
 		)
 		(property "Footprint" "PCM_Resistor_THT_AKL:R_Axial_DIN0207_L6.3mm_D2.5mm_P10.16mm_Horizontal"
-			(at 127 74.168 90)
+			(at 115.57 67.818 90)
 			(effects
 				(font
@@
 		)
 		(property "Datasheet" "~"
-			(at 127 72.39 0)
+			(at 115.57 66.04 0)
 			(effects
 				(font
@@
 		)
 		(property "Description" "Resistor"
-			(at 127 72.39 0)
+			(at 115.57 66.04 0)
 			(effects
 				(font
@@
 	(symbol
 		(lib_id "power:+3.3V")
-		(at 132.08 72.39 0)
+		(at 111.76 66.04 0)
 		(unit 1)
 		(exclude_from_sim no)
@@
 		(fields_autoplaced yes)
 		(property "Reference" "#PWR049"
-			(at 132.08 76.2 0)
+			(at 111.76 69.85 0)
 			(effects
 				(font
@@
 		)
 		(property "Value" "+3.3V"
-			(at 132.08 67.31 0)
+			(at 111.76 60.96 0)
 			(effects
 				(font
@@
 		)
 		(property "Footprint" ""
-			(at 132.08 72.39 0)
+			(at 111.76 66.04 0)
 			(effects
 				(font
@@
 		)
 		(property "Datasheet" ""
-			(at 132.08 72.39 0)
+			(at 111.76 66.04 0)
 			(effects
 				(font
@@
 		)
 		(property "Description" "Power symbol creates a global label with name \"+3.3V\""
-			(at 132.08 72.39 0)
+			(at 111.76 66.04 0)
 			(effects
 				(font

Commit message: fixed barrel jack
Connections:
- net +VCC: now also J9.1; no longer J9.2
- net GND: now also J9.2; no longer J9.1

Commit message: updates
Parts:
- J3, J4, J5, J6: footprint Connector_JST:JST_PH_S3B-PH-K_1x03_P2.00mm_Horizontal -> TerminalBlock_Phoenix:TerminalBlock_Phoenix_MPT-0,5-3-2.54_1x03_P2.54mm_Horizontal
Changed lines of the file:
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@@
 			)
 		)
-		(property "Footprint" "Connector_JST:JST_PH_S3B-PH-K_1x03_P2.00mm_Horizontal"
+		(property "Footprint" "TerminalBlock_Phoenix:TerminalBlock_Phoenix_MPT-0,5-3-2.54_1x03_P2.54mm_Horizontal"
 			(at 224.79 83.82 0)
 			(effects
@@
 			)
 		)
-		(property "Footprint" "Connector_JST:JST_PH_S3B-PH-K_1x03_P2.00mm_Horizontal"
+		(property "Footprint" "TerminalBlock_Phoenix:TerminalBlock_Phoenix_MPT-0,5-3-2.54_1x03_P2.54mm_Horizontal"
 			(at 226.06 153.67 0)
 			(effects
@@
 			)
 		)
-		(property "Footprint" "Connector_JST:JST_PH_S3B-PH-K_1x03_P2.00mm_Horizontal"
+		(property "Footprint" "TerminalBlock_Phoenix:TerminalBlock_Phoenix_MPT-0,5-3-2.54_1x03_P2.54mm_Horizontal"
 			(at 224.79 105.41 0)
 			(effects
@@
 			)
 		)
-		(property "Footprint" "Connector_JST:JST_PH_S3B-PH-K_1x03_P2.00mm_Horizontal"
+		(property "Footprint" "TerminalBlock_Phoenix:TerminalBlock_Phoenix_MPT-0,5-3-2.54_1x03_P2.54mm_Horizontal"
 			(at 224.79 127 0)
 			(effects
